Commit message: feat: urdf.xacro that assemble all the sensors of the magnet_v2.

File: urdf/magnet_v2.urdf.xacro (robot description, xacro)
@@ -1,80 +1,78 @@
 <?xml version="1.0"?>
 <robot xmlns:xacro="http://www.ros.org/wiki/xacro" name="magnet_v2">
-  <xacro:macro name="magnet_v2" params="parent *origin prefix:='' name:=magnet_v2
-                                     simulation:=false use_gpu:=true">
-    <joint name="${parent}_to_${prefix}magnet_v2_top_case" type="fixed">
+  <xacro:macro name="magnet_v2" params="parent *origin prefix:='' name:=magnet_v2 simulation:=false use_gpu:=true">
+    <xacro:property name="imu_base_height" value="0.1115"/>
+    <link name="${prefix}magnet_v2_base_mount" />
+    <joint name="${parent}_to_${prefix}magnet_v2_base_mount" type="fixed">
       <xacro:insert_block name="origin"/>
       <parent link="${parent}" />
-      <child link="${prefix}magnet_v2_top_case" />
+      <child link="${prefix}magnet_v2_base_mount" />
     </joint>
-    <link name="${prefix}magnet_v2_top_case">
+    <joint name="${prefix}magnet_v2_base_mount_to_${prefix}magnet_v2_heatsink_and_case" type="fixed">
+      <parent link="${prefix}magnet_v2_base_mount" />
+      <child link="${prefix}magnet_v2_heatsink_and_case" />
+      <origin xyz="0 0 ${imu_base_height}" rpy="0 0 0" />
+    </joint>
+    <link name="${prefix}magnet_v2_heatsink_and_case">
       <visual>
         <material name="darkgrey">
-            <color rgba="0.3 0.3 0.3 1"/>
+          <color rgba="0.3 0.3 0.3 1"/>
         </material>
-        <origin xyz="0 0 -0.056" rpy="${pi} 0 0"/>
+        <origin xyz="0 0 0" rpy="0 0 0"/>
         <geometry>
-          <mesh filename="package://magnet_description/meshes/visual/top case v3.stl" scale="0.001 0.001 0.001"/>
+          <mesh filename="package://magnet_v2_description/meshes/visual/magnet_v2_heatsink_and_case.STL" scale="1 1 1"/>
         </geometry>
       </visual>
     </link>
-    <xacro:include filename="$(find microstrain_inertial_description)/urdf/gx5_ar.urdf.xacro"/>
-    <xacro:gx5_ar name="${prefix}gx5_ar" parent="${prefix}magnet_v2_top_case">
-      <origin xyz="0.00 0.0 0.0" rpy="0 0 0" />
-    </xacro:gx5_ar>
-    <xacro:include filename="$(find E-con_inertial_description)/urdf/E-con_eCAM.urdf.xacro"/>
-    <xacro:E-con_eCAM name="${prefix}left_camera" parent="${prefix}magnet_v2_top_case">
-      <origin xyz="0.00 0.043 -0.011" rpy="0 0 ${pi/2}" />
-    </xacro:left_E-con>
-    <xacro:E-con_eCAM name="${prefix}centre_camera" parent="${prefix}magnet_v2_top_case">
-      <origin xyz="-0.043 0.000 -0.011" rpy="0 0 0" />
-    </xacro:E-con_eCAM>
-    <xacro:E-con_eCAM name="${prefix}right_camera" parent="${prefix}magnet_v2_top_case">
-      <origin xyz="0.00 -0.043 -0.011" rpy="0 0 ${-pi/2}" />
-    </xacro:E-con_eCAM>
-    <link name="heatsink">
+    <link name="${prefix}left_camera">
       <visual>
-        <material name="silver">
-            <color rgba="0.7 0.7 0.7 1"/>
-        </material>
-        <origin xyz="0 0 0.01" rpy="${pi} 0 0"/>
+        <origin xyz="0 0 0" rpy="0 0 0"/>
         <geometry>
-          <mesh filename="package://magnet_v2_description/meshes/visual/heatsink lidar v2.stl" scale="0.001 0.001 0.001"/>
+          <mesh filename="package://magnet_v2_description/meshes/visual/eCon_cam_Base.STL" scale="1 1 1"/>
         </geometry>
+        <material name="darkgrey"/>
       </visual>
     </link>
-    <joint name="${prefix}magnet_v2_top_case_to_${prefix}heatsink" type="fixed">
-      <origin xyz="0 0 0" rpy="0 0 0" />
-      <parent link="${prefix}magnet_v2_top_case" />
-      <child link="${prefix}heatsink" />
+    <joint name="${prefix}magnet_to_left_camera" type="fixed">
+      <parent link="${prefix}magnet_v2_heatsink_and_case"/>
+      <child link="${prefix}left_camera"/>
+      <origin xyz="0.00 -0.043 -0.011" rpy="${pi/2} ${pi} 0"/>
     </joint>
-    <link name="bottom_case">
+    <link name="${prefix}centre_camera">
       <visual>
-        <material name="darkgrey">
-            <color rgba="0.3 0.3 0.3 1"/>
-        </material>
-        <origin xyz="0 0 -0.056" rpy="${pi} 0 0"/>
+        <origin xyz="0 0 0" rpy="0 0 0"/>
         <geometry>
-          <mesh filename="package://magnet_v2_description/meshes/visual/bottom case v3.stl" scale="0.001 0.001 0.001"/>
+          <mesh filename="package://magnet_v2_description/meshes/visual/eCon_cam_Base.STL" scale="1 1 1"/>
         </geometry>
+        <material name="darkgrey"/>
       </visual>
     </link>
-    <joint name="${prefix}magnet_v2_top_case_to_${prefix}bottom_case" type="fixed">
-      <origin xyz="0 0 0" rpy="0 0 0" />
-      <parent link="${prefix}magnet_v2_top_case" />
-      <child link="${prefix}bottom_case" />
+    <joint name="${prefix}magnet_to_centre_camera" type="fixed">
+      <parent link="${prefix}magnet_v2_heatsink_and_case"/>
+      <child link="${prefix}centre_camera"/>
+      <origin xyz="-0.043 0.000 -0.011" rpy="${-pi/2} 0 ${pi/2}"/>
     </joint>
+    <link name="${prefix}right_camera">
+      <visual>
+        <origin xyz="0 0 0" rpy="0 0 0"/>
+        <geometry>
+          <mesh filename="package://magnet_v2_description/meshes/visual/eCon_cam_Base.STL" scale="1 1 1"/>
+        </geometry>
+        <material name="darkgrey"/>
+      </visual>
+    </link>
+    <joint name="${prefix}magnet_to_right_camera" type="fixed">
+      <parent link="${prefix}magnet_v2_heatsink_and_case"/>
+      <child link="${prefix}right_camera"/>
+      <origin xyz="0.000 0.043 -0.011" rpy="${-pi/2} 0 0"/>
+    </joint>
+    <xacro:include filename="$(find microstrain_inertial_description)/urdf/gx5_25.urdf.xacro"/>
+    <xacro:gx5_25 name="${prefix}gx5_25" parent="${prefix}magnet_v2_heatsink_and_case">
+      <origin xyz="0.00 0.0 0.0" rpy="${pi} 0 0" />
+    </xacro:gx5_25>
     <xacro:include filename="$(find hesai_description)/urdf/hesai_qt64.urdf.xacro"/>
-    <!-- The height of the Magnet 3D-printed case: From bottom of case to the origin of the imu -->
-    <xacro:property name="magnet_case_height" value="0.11512"/>
-    <xacro:hesai_qt64 name="${prefix}hesai_qt64" parent="${prefix}magnet_v2_top_case" simulation="${simulation}" use_gpu="${use_gpu}">
-      <origin xyz="0 0 0.01" rpy="0 0 0" />
-    </xacro:hesai_qt64>
-    <link name="${prefix}magnet_v2_base" />
-    <joint name="${prefix}magnet_v2_top_case_to_${prefix}magnet_base" type="fixed">
-      <parent link="${prefix}magnet_v2_top_case" />
-      <child link="${prefix}magnet_v2_base" />
-      <origin xyz="0 0 ${magnet_v2_case_height}" rpy="0 0 0" />
-    </joint>
+    <xacro:hesai_qt64_device name="${prefix}hesai_qt64_device" parent="${prefix}magnet_v2_heatsink_and_case" simulation="${simulation}" use_gpu="${use_gpu}">
+      <origin xyz="0 0 0.01" rpy="0 0 ${pi}" />
+    </xacro:hesai_qt64_device>
   </xacro:macro>
 </robot>

Commit message: do nothing

File: urdf/magnet_v2.urdf.xacro (robot description, xacro)
@@ -19,12 +19,12 @@
       </visual>
     </link>
-    <xacro:include filename="$(find microstrain_inertial_description)/urdf/gx5_ar.urdf.xacro"/>
-    <xacro:gx5_ar name="${prefix}gx5_ar" parent="${prefix}magnet_v2_top_case">
+    <xacro:include filename="$(find microstrain_inertial_description)/urdf/gx5_25.urdf.xacro"/>
+    <xacro:gx5_25 name="${prefix}gx5_ar" parent="${prefix}magnet_v2_top_case">
       <origin xyz="0.00 0.0 0.0" rpy="0 0 0" />
-    </xacro:gx5_ar>
-    <xacro:include filename="$(find E-con_inertial_description)/urdf/E-con_eCAM.urdf.xacro"/>
+    </xacro:gx5_25>
+    <!-- <xacro:include filename="$(find E-con_inertial_description)/urdf/E-con_eCAM.urdf.xacro"/>
     <xacro:E-con_eCAM name="${prefix}left_camera" parent="${prefix}magnet_v2_top_case">
       <origin xyz="0.00 0.043 -0.011" rpy="0 0 ${pi/2}" />
-    </xacro:left_E-con>
+    </xacro:E-con_eCAM>
     <xacro:E-con_eCAM name="${prefix}centre_camera" parent="${prefix}magnet_v2_top_case">
       <origin xyz="-0.043 0.000 -0.011" rpy="0 0 0" />
@@ -32,5 +32,5 @@
     <xacro:E-con_eCAM name="${prefix}right_camera" parent="${prefix}magnet_v2_top_case">
       <origin xyz="0.00 -0.043 -0.011" rpy="0 0 ${-pi/2}" />
-    </xacro:E-con_eCAM>
+    </xacro:E-con_eCAM> -->
     <link name="heatsink">
       <visual>
@@ -67,5 +67,5 @@
     <xacro:include filename="$(find hesai_description)/urdf/hesai_qt64.urdf.xacro"/>
     <!-- The height of the Magnet 3D-printed case: From bottom of case to the origin of the imu -->
-    <xacro:property name="magnet_case_height" value="0.11512"/>
+    <xacro:property name="magnet_v2_case_height" value="0.11512"/>
     <xacro:hesai_qt64 name="${prefix}hesai_qt64" parent="${prefix}magnet_v2_top_case" simulation="${simulation}" use_gpu="${use_gpu}">
       <origin xyz="0 0 0.01" rpy="0 0 0" />

Commit message: feat: 1) Change tp make the root, magnet_mount +x forward 2) add new link of magnet_base, +x facing forward

File: urdf/magnet_v2.urdf.xacro (robot description, xacro)
@@ -3,16 +3,16 @@
   <xacro:macro name="magnet_v2" params="parent *origin prefix:='' name:=magnet_v2 simulation:=false use_gpu:=true">
     <xacro:property name="imu_base_height" value="0.1115"/>
-    <link name="${prefix}magnet_v2_base_mount" />
-    <joint name="${parent}_to_${prefix}magnet_v2_base_mount" type="fixed">
+    <link name="${prefix}magnet_mount" />
+    <joint name="${parent}_to_${prefix}magnet_mount" type="fixed">
       <xacro:insert_block name="origin"/>
       <parent link="${parent}" />
-      <child link="${prefix}magnet_v2_base_mount" />
+      <child link="${prefix}magnet_mount" />
     </joint>
-    <joint name="${prefix}magnet_v2_base_mount_to_${prefix}magnet_v2_heatsink_and_case" type="fixed">
-      <parent link="${prefix}magnet_v2_base_mount" />
-      <child link="${prefix}magnet_v2_heatsink_and_case" />
-      <origin xyz="0 0 ${imu_base_height}" rpy="0 0 0" />
+    <joint name="${prefix}magnet_mount_to_${prefix}magnet_case" type="fixed">
+      <parent link="${prefix}magnet_mount" />
+      <child link="${prefix}magnet_case" />
+      <origin xyz="0 0 ${imu_base_height}" rpy="0 0 ${pi}" />
     </joint>
-    <link name="${prefix}magnet_v2_heatsink_and_case">
+    <link name="${prefix}magnet_case">
       <visual>
         <material name="darkgrey">
@@ -35,5 +35,5 @@
     </link>
     <joint name="${prefix}magnet_to_left_camera" type="fixed">
-      <parent link="${prefix}magnet_v2_heatsink_and_case"/>
+      <parent link="${prefix}magnet_case"/>
       <child link="${prefix}left_camera"/>
       <origin xyz="0.00 -0.043 -0.011" rpy="${pi/2} ${pi} 0"/>
@@ -49,5 +49,5 @@
     </link>
     <joint name="${prefix}magnet_to_centre_camera" type="fixed">
-      <parent link="${prefix}magnet_v2_heatsink_and_case"/>
+      <parent link="${prefix}magnet_case"/>
       <child link="${prefix}centre_camera"/>
       <origin xyz="-0.043 0.000 -0.011" rpy="${-pi/2} 0 ${pi/2}"/>
@@ -63,14 +63,20 @@
     </link>
     <joint name="${prefix}magnet_to_right_camera" type="fixed">
-      <parent link="${prefix}magnet_v2_heatsink_and_case"/>
+      <parent link="${prefix}magnet_case"/>
       <child link="${prefix}right_camera"/>
       <origin xyz="0.000 0.043 -0.011" rpy="${-pi/2} 0 0"/>
     </joint>
     <xacro:include filename="$(find microstrain_inertial_description)/urdf/gx5_25.urdf.xacro"/>
-    <xacro:gx5_25 name="${prefix}gx5_25" parent="${prefix}magnet_v2_heatsink_and_case">
+    <xacro:gx5_25 name="${prefix}gx5_25" parent="${prefix}magnet_case">
       <origin xyz="0.00 0.0 0.0" rpy="${pi} 0 0" />
     </xacro:gx5_25>
+    <link name="${prefix}magnet_base" />
+    <joint name="${prefix}magnet_case_to_${prefix}magnet_base" type="fixed">
+      <parent link="${prefix}magnet_case" />
+      <child link="${prefix}magnet_base" />
+      <origin xyz="0 0 0.01" rpy="0 0 ${pi}" />
+    </joint>
     <xacro:include filename="$(find hesai_description)/urdf/hesai_qt64.urdf.xacro"/>
-    <xacro:hesai_qt64_device name="${prefix}hesai_qt64_device" parent="${prefix}magnet_v2_heatsink_and_case" simulation="${simulation}" lidar_frame="hesai_lidar" use_gpu="${use_gpu}">
+    <xacro:hesai_qt64_device name="${prefix}hesai_qt64_device" parent="${prefix}magnet_case" simulation="${simulation}" lidar_frame="hesai_lidar" use_gpu="${use_gpu}">
       <origin xyz="0 0 0.01" rpy="0 0 ${pi}" />
     </xacro:hesai_qt64_device>

Commit message: feat: 1) Change tp make the root, magnet_mount +x forward 2) add new link of magnet_base, +x facing forward

File: urdf/magnet_v2.urdf.xacro (robot description, xacro)
@@ -3,16 +3,16 @@
   <xacro:macro name="magnet_v2" params="parent *origin prefix:='' name:=magnet_v2 simulation:=false use_gpu:=true">
     <xacro:property name="imu_base_height" value="0.1115"/>
-    <link name="${prefix}magnet_v2_base_mount" />
-    <joint name="${parent}_to_${prefix}magnet_v2_base_mount" type="fixed">
+    <link name="${prefix}magnet_mount" />
+    <joint name="${parent}_to_${prefix}magnet_mount" type="fixed">
       <xacro:insert_block name="origin"/>
       <parent link="${parent}" />
-      <child link="${prefix}magnet_v2_base_mount" />
+      <child link="${prefix}magnet_mount" />
     </joint>
-    <joint name="${prefix}magnet_v2_base_mount_to_${prefix}magnet_v2_heatsink_and_case" type="fixed">
-      <parent link="${prefix}magnet_v2_base_mount" />
-      <child link="${prefix}magnet_v2_heatsink_and_case" />
-      <origin xyz="0 0 ${imu_base_height}" rpy="0 0 0" />
+    <joint name="${prefix}magnet_mount_to_${prefix}magnet_case" type="fixed">
+      <parent link="${prefix}magnet_mount" />
+      <child link="${prefix}magnet_case" />
+      <origin xyz="0 0 ${imu_base_height}" rpy="0 0 ${pi}" />
     </joint>
-    <link name="${prefix}magnet_v2_heatsink_and_case">
+    <link name="${prefix}magnet_case">
       <visual>
         <material name="darkgrey">
@@ -35,5 +35,5 @@
     </link>
     <joint name="${prefix}magnet_to_left_camera" type="fixed">
-      <parent link="${prefix}magnet_v2_heatsink_and_case"/>
+      <parent link="${prefix}magnet_case"/>
       <child link="${prefix}left_camera"/>
       <origin xyz="0.00 -0.043 -0.011" rpy="${pi/2} ${pi} 0"/>
@@ -49,5 +49,5 @@
     </link>
     <joint name="${prefix}magnet_to_centre_camera" type="fixed">
-      <parent link="${prefix}magnet_v2_heatsink_and_case"/>
+      <parent link="${prefix}magnet_case"/>
       <child link="${prefix}centre_camera"/>
       <origin xyz="-0.043 0.000 -0.011" rpy="${-pi/2} 0 ${pi/2}"/>
@@ -63,14 +63,20 @@
     </link>
     <joint name="${prefix}magnet_to_right_camera" type="fixed">
-      <parent link="${prefix}magnet_v2_heatsink_and_case"/>
+      <parent link="${prefix}magnet_case"/>
       <child link="${prefix}right_camera"/>
       <origin xyz="0.000 0.043 -0.011" rpy="${-pi/2} 0 0"/>
     </joint>
     <xacro:include filename="$(find microstrain_inertial_description)/urdf/gx5_25.urdf.xacro"/>
-    <xacro:gx5_25 name="${prefix}gx5_25" parent="${prefix}magnet_v2_heatsink_and_case">
+    <xacro:gx5_25 name="${prefix}gx5_25" parent="${prefix}magnet_case">
       <origin xyz="0.00 0.0 0.0" rpy="${pi} 0 0" />
     </xacro:gx5_25>
+    <link name="${prefix}magnet_base" />
+    <joint name="${prefix}magnet_case_to_${prefix}magnet_base" type="fixed">
+      <parent link="${prefix}magnet_case" />
+      <child link="${prefix}magnet_base" />
+      <origin xyz="0 0 0.01" rpy="0 0 ${pi}" />
+    </joint>
     <xacro:include filename="$(find hesai_description)/urdf/hesai_qt64.urdf.xacro"/>
-    <xacro:hesai_qt64 name="${prefix}hesai_qt64_device" parent="${prefix}magnet_v2_heatsink_and_case" simulation="${simulation}" use_gpu="${use_gpu}" lidar_frame="hesai_lidar">
+    <xacro:hesai_qt64 name="${prefix}hesai_qt64_device" parent="${prefix}magnet_case" simulation="${simulation}" use_gpu="${use_gpu}" lidar_frame="hesai_lidar">
       <origin xyz="0 0 0.01" rpy="0 0 ${pi}" />
     </xacro:hesai_qt64>
